File: pcb/left/worxboard-left.kicad_pcb (KiCad board)
At the start: 2 copper layers, 182.8 x 158.8 mm, 141 parts, among them J1 TYPE-C-31-M-12, J2 PJ-320D-4A, J3 nice!view, SW1 BOOT, SW2 RESET, U1 RP2040, U2 W25Q128JVSIQ, U3 AP2112K-3.3, U4 USBLC6-2SC6, U5 USBLC6-2SC6, Y1 12MHz

Commit message: feat(pcb): transactional rip-up completion; left board routed (DRC clean, 0 unconnected)
- complete_routes.negotiate(): soft-route an open gap across unlocked copper, rip it up,
  reroute the victims (three levels), keep the change only if fewer islands remain
- exact path check against fixed copper so stub ends 0.3 mm from a via can escape
- delete copper with BOARD.Delete (Remove + GC corrupted the board under SWIG)
- drop Freerouting tracks below the 0.127 mm board minimum before completion
- left half: no B.Cu USB keepout across U4, so its VBUS via can leave

Co-Authored-By: Claude Opus 5.5 <noreply@anthropic.com>
Routing:
- net ROW5: track 105.1 -> 258.7 mm, vias 8 -> 15
- net COL5: track 112.6 -> 229.6 mm, vias 9 -> 15
- net COL4: track 165.1 -> 250.9 mm, vias 8 -> 14
- net DISP_DC: track 6.65 -> 84.8 mm, vias 1 -> 2
- net 1V1: track 22.1 -> 90.7 mm, vias 2 -> 13
- net VBUS: track 68.2 -> 30.1 mm, vias 5 -> 3
- net 3V3: track 258.2 -> 284.2 mm, vias 8 -> 17
- net COL6: track 203.6 -> 223.4 mm, vias 10 -> 8
- net COL1: track 231.8 -> 213.1 mm, vias 14 -> 9
- net COL0: track 149.7 -> 136.0 mm, vias 6 -> 8
- net QSPI_SS: track 23.2 -> 35.8 mm, vias 4 -> 7
- net COL3: track 237.9 -> 248.8 mm, vias 10 -> 14
- net RUN: track 29.9 -> 39.1 mm, vias 2 -> 4
- net QSPI_SD3: track 3.39 -> 11.9 mm, vias 0 -> 2
- net TRRS_A: track 24.9 -> 32.7 mm, vias 3 -> 2
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
Commit message: feat(pcb): route both halves to 0 unconnected (DRC + checks pass)
- negotiate: protected nets are dear rather than fixed, GND judged on a fresh fill,
  stuck nets spared on the next try, lanes kept clear ahead of locked stub ends
- pours join pads by overlap and tracks / vias only by anchor, as in KiCad
- left and right boards regenerated: 0 violations, 0 unconnected, 0 parity issues
- deviations WS2b-6 (rip-up) and WS2b-7 (left U4 keepout gap)

Co-Authored-By: Claude Opus 5.5 <noreply@anthropic.com>
Routing:
- net 1V1: track 90.7 -> 54.1 mm, vias 13 -> 7
- net ROW5: track 258.7 -> 294.3 mm, vias 15 -> 23
- net ROW4: track 207.4 -> 229.4 mm
- net XOUT: track 8.72 -> 27.7 mm, vias 2 -> 5
- net ROW3: track 234.1 -> 249.5 mm, vias 8 -> 10
- net QSPI_SS: track 35.8 -> 24.3 mm, vias 7 -> 2
- net RUN: track 39.1 -> 31.1 mm, vias 4 -> 5
- net COL2: track 223.5 -> 231.2 mm, vias 12 -> 11
- net GND: track 3.93 -> 10.4 mm, vias 102 -> 103
- net VBUS_SENSE: track 34.6 -> 28.3 mm, vias 3 -> 2
- net QSPI_SD0: track 19.4 -> 13.2 mm, vias 3 -> 2
- net CC1: track 20.0 -> 14.1 mm, vias 4 -> 2
- net COL1: track 213.1 -> 218.2 mm, vias 9 -> 12
- net COL5: track 229.6 -> 224.6 mm, vias 15 -> 17
- net 3V3: track 284.2 -> 279.5 mm, vias 17 -> 21
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
Commit message: feat(pcb): seed KIIDs and the hash seed so a clean rebuild reproduces the boards
place/route_critical/import_ses seed KiCad's UUID generator from their inputs and a
per-side base seed; pcb.just runs with PYTHONHASHSEED=0. Boards re-made from scratch
with the seeded pipeline (DRC 0 violations, 0 unconnected, checks pass), renders refreshed.

Co-Authored-By: Claude Opus 5.5 <noreply@anthropic.com>
Routing:
- net COL0: track 137.1 -> 165.0 mm
- net ROW4: track 229.4 -> 201.8 mm, vias 7 -> 16
- net COL5: track 224.6 -> 200.0 mm, vias 17 -> 11
- net ROW5: track 294.3 -> 270.0 mm, vias 23 -> 17
- net 3V3: track 279.5 -> 255.5 mm, vias 21 -> 15
- net COL4: track 250.5 -> 228.1 mm, vias 14 -> 9
- net UART_RX: track 135.1 -> 155.9 mm, vias 6 -> 9
- net GND: track 10.4 -> 28.8 mm, vias 103 -> 114
- net CC1: track 14.1 -> 31.7 mm, vias 2 -> 5
- net COL2: track 231.2 -> 213.9 mm, vias 11 -> 8
- net COL3: track 250.4 -> 233.5 mm
- net COL1: track 218.2 -> 233.4 mm, vias 12 -> 14
- net XOUT: track 27.7 -> 13.0 mm, vias 5 -> 2
- net DISP_RST: track 82.7 -> 97.4 mm, vias 2 -> 9
- net COL6: track 223.9 -> 210.0 mm, vias 9 -> 7
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